File: pcb/hmkb64alps.kicad_pcb (KiCad board)
At the start: 2 copper layers, 0 parts

Commit message: place switches and set some design rules
Parts:
- added C1: 10uF, Capacitor_SMD:C_0805_2012Metric_Pad1.18x1.45mm_HandSolder, F.Cu at (-34.7, -48.8)
- added C2: 0.1uF, Capacitor_SMD:C_0805_2012Metric_Pad1.18x1.45mm_HandSolder, F.Cu at (-34.7, -45.8)
- added C3: 0.1uF, Capacitor_SMD:C_0805_2012Metric_Pad1.18x1.45mm_HandSolder, F.Cu at (-34.7, -42.8)
- added C4: 0.1uF, Capacitor_SMD:C_0805_2012Metric_Pad1.18x1.45mm_HandSolder, F.Cu at (-34.7, -39.8)
- added C5: C_Small, Capacitor_SMD:C_0805_2012Metric_Pad1.18x1.45mm_HandSolder, F.Cu at (-34.7, -36.8)
- added C6: C_Small, Capacitor_SMD:C_0805_2012Metric_Pad1.18x1.45mm_HandSolder, F.Cu at (-34.7, -33.8)
- added C7: 0.1uF, Capacitor_SMD:C_0805_2012Metric_Pad1.18x1.45mm_HandSolder, F.Cu at (-34.7, -30.8)
- added C8: 1uF, Capacitor_SMD:C_0805_2012Metric_Pad1.18x1.45mm_HandSolder, F.Cu at (-34.7, -27.7)
- added D1: D, Diode_SMD:D_SOD-123, B.Cu at (41.5, 43.1)
- added D10: D, Diode_SMD:D_SOD-123, B.Cu at (212.9, 43.1)
- added D11: D, Diode_SMD:D_SOD-123, B.Cu at (232.0, 43.1)
- added D12: D, Diode_SMD:D_SOD-123, B.Cu at (251.1, 43.1)
- added D13: D, Diode_SMD:D_SOD-123, B.Cu at (270.1, 43.1)
- added D14: D, Diode_SMD:D_SOD-123, B.Cu at (298.7, 43.1)
- added D15: D, Diode_SMD:D_SOD-123, B.Cu at (327.2, 43.1)
- added D16: D, Diode_SMD:D_SOD-123, B.Cu at (46.3, 62.1)
- added D17: D, Diode_SMD:D_SOD-123, B.Cu at (70.1, 62.1)
- added D18: D, Diode_SMD:D_SOD-123, B.Cu at (89.1, 62.1)
- added D19: D, Diode_SMD:D_SOD-123, B.Cu at (108.2, 62.1)
- added D2: D, Diode_SMD:D_SOD-123, B.Cu at (60.5, 43.1)
- added D20: D, Diode_SMD:D_SOD-123, B.Cu at (127.2, 62.1)
- added D21: D, Diode_SMD:D_SOD-123, B.Cu at (146.3, 62.1)
- added D22: D, Diode_SMD:D_SOD-123, B.Cu at (165.3, 62.1)
- added D23: D, Diode_SMD:D_SOD-123, B.Cu at (184.4, 62.1)
- added D24: D, Diode_SMD:D_SOD-123, B.Cu at (203.4, 62.1)
- added D25: D, Diode_SMD:D_SOD-123, B.Cu at (222.5, 62.1)
- added D26: D, Diode_SMD:D_SOD-123, B.Cu at (241.5, 62.1)
- added D27: D, Diode_SMD:D_SOD-123, B.Cu at (260.6, 62.1)
- added D28: D, Diode_SMD:D_SOD-123, B.Cu at (279.6, 62.1)
- added D29: D, Diode_SMD:D_SOD-123, B.Cu at (303.4, 62.1)
- added D3: D, Diode_SMD:D_SOD-123, B.Cu at (79.6, 43.1)
- added D30: D, Diode_SMD:D_SOD-123, B.Cu at (327.2, 62.1)
- added D31: D, Diode_SMD:D_SOD-123, B.Cu at (48.6, 81.2)
- added D32: D, Diode_SMD:D_SOD-123, B.Cu at (74.8, 81.2)
- added D33: D, Diode_SMD:D_SOD-123, B.Cu at (93.9, 81.2)
- added D34: D, Diode_SMD:D_SOD-123, B.Cu at (112.9, 81.2)
- added D35: D, Diode_SMD:D_SOD-123, B.Cu at (132.0, 81.2)
- added D36: D, Diode_SMD:D_SOD-123, B.Cu at (151.0, 81.2)
- added D37: D, Diode_SMD:D_SOD-123, B.Cu at (170.1, 81.2)
- added D38: D, Diode_SMD:D_SOD-123, B.Cu at (189.1, 81.2)
- added D39: D, Diode_SMD:D_SOD-123, B.Cu at (208.2, 81.2)
- added D4: D, Diode_SMD:D_SOD-123, B.Cu at (98.7, 43.1)
- added D40: D, Diode_SMD:D_SOD-123, B.Cu at (227.2, 81.2)
- added D41: D, Diode_SMD:D_SOD-123, B.Cu at (246.3, 81.2)
- added D42: D, Diode_SMD:D_SOD-123, B.Cu at (265.3, 81.2)
- added D43: D, Diode_SMD:D_SOD-123, B.Cu at (296.3, 81.2)
- added D44: D, Diode_SMD:D_SOD-123, B.Cu at (327.2, 81.2)
- added D45: D, Diode_SMD:D_SOD-123, B.Cu at (53.4, 100.2)
- added D46: D, Diode_SMD:D_SOD-123, B.Cu at (84.4, 100.2)
- added D47: D, Diode_SMD:D_SOD-123, B.Cu at (103.4, 100.2)
- added D48: D, Diode_SMD:D_SOD-123, B.Cu at (122.5, 100.2)
- added D49: D, Diode_SMD:D_SOD-123, B.Cu at (141.5, 100.2)
- added D5: D, Diode_SMD:D_SOD-123, B.Cu at (117.7, 43.1)
- added D50: D, Diode_SMD:D_SOD-123, B.Cu at (160.6, 100.2)
- added D51: D, Diode_SMD:D_SOD-123, B.Cu at (179.6, 100.2)
- added D52: D, Diode_SMD:D_SOD-123, B.Cu at (198.7, 100.2)
- added D53: D, Diode_SMD:D_SOD-123, B.Cu at (217.7, 100.2)
- added D54: D, Diode_SMD:D_SOD-123, B.Cu at (236.8, 100.2)
- added D55: D, Diode_SMD:D_SOD-123, B.Cu at (255.8, 100.2)
- added D56: D, Diode_SMD:D_SOD-123, B.Cu at (282.0, 100.2)
- added D57: D, Diode_SMD:D_SOD-123, B.Cu at (308.2, 100.2)
- added D58: D, Diode_SMD:D_SOD-123, B.Cu at (327.2, 100.2)
- added D59: D, Diode_SMD:D_SOD-123, B.Cu at (43.9, 119.3)
- added D6: D, Diode_SMD:D_SOD-123, B.Cu at (136.8, 43.1)
- added D60: D, Diode_SMD:D_SOD-123, B.Cu at (67.7, 119.3)
- added D61: D, Diode_SMD:D_SOD-123, B.Cu at (91.5, 119.3)
- added D62: D, Diode_SMD:D_SOD-123, B.Cu at (162.9, 119.3)
- added D63: D, Diode_SMD:D_SOD-123, B.Cu at (232.0, 119.3)
- added D64: D, Diode_SMD:D_SOD-123, B.Cu at (251.1, 119.3)
- added D65: D, Diode_SMD:D_SOD-123, B.Cu at (270.1, 119.3)
- added D66: D, Diode_SMD:D_SOD-123, B.Cu at (289.1, 119.3)
- added D67: D, Diode_SMD:D_SOD-123, B.Cu at (308.2, 119.3)
- added D68: D, Diode_SMD:D_SOD-123, B.Cu at (327.2, 119.3)
- added D69: PRTR5V0U2X, Package_TO_SOT_SMD:SOT-143, B.Cu at (-7.42, -31.6)
- added D7: D, Diode_SMD:D_SOD-123, B.Cu at (155.8, 43.1)
- added D8: D, Diode_SMD:D_SOD-123, B.Cu at (174.8, 43.1)
- added D9: D, Diode_SMD:D_SOD-123, B.Cu at (193.9, 43.1)
- added F1: 500m, Fuse:Fuse_1206_3216Metric_Pad1.42x1.75mm_HandSolder, F.Cu at (-10.2, -25.7)
- added J1: AVR-ISP-6, Connector_IDC:IDC-Header_2x03_P2.54mm_Vertical, F.Cu at (-22.3, -44.2)
- added R1: 10k, Resistor_SMD:R_0805_2012Metric_Pad1.20x1.40mm_HandSolder, F.Cu at (-30.0, -48.8)
- added R2: 22, Resistor_SMD:R_0805_2012Metric_Pad1.20x1.40mm_HandSolder, F.Cu at (-30.0, -45.9)
- added R3: 22, Resistor_SMD:R_0805_2012Metric_Pad1.20x1.40mm_HandSolder, F.Cu at (-30.0, -42.9)
- added R4: 10k, Resistor_SMD:R_0805_2012Metric_Pad1.20x1.40mm_HandSolder, F.Cu at (-30.0, -40.0)
- added R5: 5.1k, Resistor_SMD:R_0805_2012Metric_Pad1.20x1.40mm_HandSolder, F.Cu at (-30.0, -37.0)
- added R6: 5.1k, Resistor_SMD:R_0805_2012Metric_Pad1.20x1.40mm_HandSolder, F.Cu at (-30.0, -34.1)
- added SW1: SW_Push, MX_Alps_Hybrid:MX-Alps-Hybrid-1U, F.Cu at (38.1, 38.1)
- added SW10: SW_Push, MX_Alps_Hybrid:MX-Alps-Hybrid-1U, F.Cu at (209.6, 38.1)
- added SW11: SW_Push, MX_Alps_Hybrid:MX-Alps-Hybrid-1U, F.Cu at (228.6, 38.1)
- added SW12: SW_Push, MX_Alps_Hybrid:MX-Alps-Hybrid-1U, F.Cu at (247.7, 38.1)
- added SW13: SW_Push, MX_Alps_Hybrid:MX-Alps-Hybrid-1U, F.Cu at (266.7, 38.1)
- added SW14: SW_Push, MX_Alps_Hybrid:MX-Alps-Hybrid-2U, F.Cu at (295.3, 38.1)
- added SW15: SW_Push, MX_Alps_Hybrid:MX-Alps-Hybrid-1U, F.Cu at (323.9, 38.1)
- added SW16: SW_Push, MX_Alps_Hybrid:MX-Alps-Hybrid-1.5U, F.Cu at (42.9, 57.1)
- added SW17: SW_Push, MX_Alps_Hybrid:MX-Alps-Hybrid-1U, F.Cu at (66.7, 57.1)
- added SW18: SW_Push, MX_Alps_Hybrid:MX-Alps-Hybrid-1U, F.Cu at (85.7, 57.1)
- added SW19: SW_Push, MX_Alps_Hybrid:MX-Alps-Hybrid-1U, F.Cu at (104.8, 57.1)
- added SW2: SW_Push, MX_Alps_Hybrid:MX-Alps-Hybrid-1U, F.Cu at (57.1, 38.1)
- added SW20: SW_Push, MX_Alps_Hybrid:MX-Alps-Hybrid-1U, F.Cu at (123.8, 57.1)
- added SW21: SW_Push, MX_Alps_Hybrid:MX-Alps-Hybrid-1U, F.Cu at (142.9, 57.1)
- added SW22: SW_Push, MX_Alps_Hybrid:MX-Alps-Hybrid-1U, F.Cu at (161.9, 57.1)
- added SW23: SW_Push, MX_Alps_Hybrid:MX-Alps-Hybrid-1U, F.Cu at (181.0, 57.1)
- added SW24: SW_Push, MX_Alps_Hybrid:MX-Alps-Hybrid-1U, F.Cu at (200.0, 57.1)
- added SW25: SW_Push, MX_Alps_Hybrid:MX-Alps-Hybrid-1U, F.Cu at (219.1, 57.1)
- added SW26: SW_Push, MX_Alps_Hybrid:MX-Alps-Hybrid-1U, F.Cu at (238.1, 57.1)
- added SW27: SW_Push, MX_Alps_Hybrid:MX-Alps-Hybrid-1U, F.Cu at (257.2, 57.1)
- added SW28: SW_Push, MX_Alps_Hybrid:MX-Alps-Hybrid-1U, F.Cu at (276.2, 57.1)
- added SW29: SW_Push, MX_Alps_Hybrid:MX-Alps-Hybrid-1.5U, F.Cu at (300.0, 57.1)
- added SW3: SW_Push, MX_Alps_Hybrid:MX-Alps-Hybrid-1U, F.Cu at (76.2, 38.1)
- added SW30: SW_Push, MX_Alps_Hybrid:MX-Alps-Hybrid-1U, F.Cu at (323.9, 57.1)
- added SW31: SW_Push, MX_Alps_Hybrid:MX-Alps-Hybrid-1.75U, F.Cu at (45.2, 76.2)
- added SW32: SW_Push, MX_Alps_Hybrid:MX-Alps-Hybrid-1U, F.Cu at (71.4, 76.2)
- added SW33: SW_Push, MX_Alps_Hybrid:MX-Alps-Hybrid-1U, F.Cu at (90.5, 76.2)
- added SW34: SW_Push, MX_Alps_Hybrid:MX-Alps-Hybrid-1U, F.Cu at (109.5, 76.2)
- added SW35: SW_Push, MX_Alps_Hybrid:MX-Alps-Hybrid-1U, F.Cu at (128.6, 76.2)
- added SW36: SW_Push, MX_Alps_Hybrid:MX-Alps-Hybrid-1U, F.Cu at (147.6, 76.2)
- added SW37: SW_Push, MX_Alps_Hybrid:MX-Alps-Hybrid-1U, F.Cu at (166.7, 76.2)
- added SW38: SW_Push, MX_Alps_Hybrid:MX-Alps-Hybrid-1U, F.Cu at (185.7, 76.2)
- added SW39: SW_Push, MX_Alps_Hybrid:MX-Alps-Hybrid-1U, F.Cu at (204.8, 76.2)
- added SW4: SW_Push, MX_Alps_Hybrid:MX-Alps-Hybrid-1U, F.Cu at (95.2, 38.1)
- added SW40: SW_Push, MX_Alps_Hybrid:MX-Alps-Hybrid-1U, F.Cu at (223.8, 76.2)
- added SW41: SW_Push, MX_Alps_Hybrid:MX-Alps-Hybrid-1U, F.Cu at (242.9, 76.2)
- added SW42: SW_Push, MX_Alps_Hybrid:MX-Alps-Hybrid-1U, F.Cu at (261.9, 76.2)
- added SW43: SW_Push, MX_Alps_Hybrid:MX-Alps-Hybrid-2.25U, F.Cu at (292.9, 76.2)
- added SW44: SW_Push, MX_Alps_Hybrid:MX-Alps-Hybrid-1U, F.Cu at (323.9, 76.2)
- added SW45: SW_Push, MX_Alps_Hybrid:MX-Alps-Hybrid-2.25U, F.Cu at (50.0, 95.2)
- added SW46: SW_Push, MX_Alps_Hybrid:MX-Alps-Hybrid-1U, F.Cu at (81.0, 95.2)
- added SW47: SW_Push, MX_Alps_Hybrid:MX-Alps-Hybrid-1U, F.Cu at (100.0, 95.2)
- added SW48: SW_Push, MX_Alps_Hybrid:MX-Alps-Hybrid-1U, F.Cu at (119.1, 95.2)
- added SW49: SW_Push, MX_Alps_Hybrid:MX-Alps-Hybrid-1U, F.Cu at (138.1, 95.2)
- added SW5: SW_Push, MX_Alps_Hybrid:MX-Alps-Hybrid-1U, F.Cu at (114.3, 38.1)
- added SW50: SW_Push, MX_Alps_Hybrid:MX-Alps-Hybrid-1U, F.Cu at (157.2, 95.2)
- added SW51: SW_Push, MX_Alps_Hybrid:MX-Alps-Hybrid-1U, F.Cu at (176.2, 95.2)
- added SW52: SW_Push, MX_Alps_Hybrid:MX-Alps-Hybrid-1U, F.Cu at (195.3, 95.2)
- added SW53: SW_Push, MX_Alps_Hybrid:MX-Alps-Hybrid-1U, F.Cu at (214.3, 95.2)
- added SW54: SW_Push, MX_Alps_Hybrid:MX-Alps-Hybrid-1U, F.Cu at (233.4, 95.2)
- added SW55: SW_Push, MX_Alps_Hybrid:MX-Alps-Hybrid-1U, F.Cu at (252.4, 95.2)
- added SW56: SW_Push, MX_Alps_Hybrid:MX-Alps-Hybrid-1.75U, F.Cu at (278.6, 95.2)
- added SW57: SW_Push, MX_Alps_Hybrid:MX-Alps-Hybrid-1U, F.Cu at (304.8, 95.2)
- added SW58: SW_Push, MX_Alps_Hybrid:MX-Alps-Hybrid-1U, F.Cu at (323.9, 95.2)
- added SW59: SW_Push, MX_Alps_Hybrid:MX-Alps-Hybrid-1.25U, F.Cu at (40.5, 114.3)
- added SW6: SW_Push, MX_Alps_Hybrid:MX-Alps-Hybrid-1U, F.Cu at (133.3, 38.1)
- added SW60: SW_Push, MX_Alps_Hybrid:MX-Alps-Hybrid-1.25U, F.Cu at (64.3, 114.3)
- added SW61: SW_Push, MX_Alps_Hybrid:MX-Alps-Hybrid-1.25U, F.Cu at (88.1, 114.3)
- added SW62: SW_Push, MX_Alps_Hybrid:MX-Alps-Hybrid-6.25U, F.Cu at (159.5, 114.3)
- added SW63: SW_Push, MX_Alps_Hybrid:MX-Alps-Hybrid-1U, F.Cu at (228.6, 114.3)
- added SW64: SW_Push, MX_Alps_Hybrid:MX-Alps-Hybrid-1U, F.Cu at (247.7, 114.3)
- added SW65: SW_Push, MX_Alps_Hybrid:MX-Alps-Hybrid-1U, F.Cu at (266.7, 114.3)
- added SW66: SW_Push, MX_Alps_Hybrid:MX-Alps-Hybrid-1U, F.Cu at (285.8, 114.3)
- added SW67: SW_Push, MX_Alps_Hybrid:MX-Alps-Hybrid-1U, F.Cu at (304.8, 114.3)
- added SW68: SW_Push, MX_Alps_Hybrid:MX-Alps-Hybrid-1U, F.Cu at (323.9, 114.3)
- added SW69: SW_Push, Button_Switch_SMD:SW_SPST_SKQG_WithStem, F.Cu at (-10.8, -36.6)
- added SW7: SW_Push, MX_Alps_Hybrid:MX-Alps-Hybrid-1U, F.Cu at (152.4, 38.1)
- added SW8: SW_Push, MX_Alps_Hybrid:MX-Alps-Hybrid-1U, F.Cu at (171.4, 38.1)
- added SW9: SW_Push, MX_Alps_Hybrid:MX-Alps-Hybrid-1U, F.Cu at (190.5, 38.1)
- added U1: ATmega32U4-A, Package_QFP:TQFP-44_10x10mm_P0.8mm, F.Cu at (-20.4, -25.8)
- added USB1: GCT USB-C USB4085-GF-A, ai03-2725_Type-C:USB_C_GCT_USB4085, F.Cu at (-10.3, -43.1)
- added Y1: 16MHz, Crystal:Crystal_SMD_3225-4Pin_3.2x2.5mm_HandSoldering, F.Cu at (-9.80, -30.1)
Routing:
- net ROW1: track 0.00 -> 281.0 mm
- net ROW3: track 0.00 -> 242.9 mm
- net ROW0: track 0.00 -> 228.6 mm
- net ROW2: track 0.00 -> 216.7 mm
- net ROW4: track 0.00 -> 142.9 mm
- net COL2: track 0.00 -> 89.0 mm
- net COL5: track 0.00 -> 87.0 mm
- net COL9: track 0.00 -> 86.0 mm
- net COL10: track 0.00 -> 86.0 mm
- net COL12: track 0.00 -> 84.1 mm
- net COL11: track 0.00 -> 84.1 mm
- net COL0: track 0.00 -> 83.1 mm
- net COL14: track 0.00 -> 76.2 mm
- net COL6: track 0.00 -> 67.0 mm
- net COL4: track 0.00 -> 67.0 mm
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