File: pcb/hmkb64alps.kicad_pcb (KiCad board)
At the start: 2 copper layers, 157 parts, among them J1 AVR-ISP-6, SW1 SW_Push, SW10 SW_Push, SW11 SW_Push, SW12 SW_Push, SW13 SW_Push, SW14 SW_Push, SW15 SW_Push, SW16 SW_Push, SW17 SW_Push, SW18 SW_Push, SW19 SW_Push, SW2 SW_Push, SW20 SW_Push, SW21 SW_Push, SW22 SW_Push, SW23 SW_Push, SW24 SW_Push, SW25 SW_Push, SW26 SW_Push, SW27 SW_Push, SW28 SW_Push, SW29 SW_Push, SW3 SW_Push, SW30 SW_Push, SW31 SW_Push, SW32 SW_Push, SW33 SW_Push, SW34 SW_Push, SW35 SW_Push, SW36 SW_Push, SW37 SW_Push, SW38 SW_Push, SW39 SW_Push, SW4 SW_Push, SW40 SW_Push, SW41 SW_Push, SW42 SW_Push, SW43 SW_Push, SW44 SW_Push, SW45 SW_Push, SW46 SW_Push, SW47 SW_Push, SW48 SW_Push, SW49 SW_Push, SW5 SW_Push, SW50 SW_Push, SW51 SW_Push, SW52 SW_Push, SW53 SW_Push, SW54 SW_Push, SW55 SW_Push, SW56 SW_Push, SW57 SW_Push, SW58 SW_Push, SW59 SW_Push, SW6 SW_Push, SW60 SW_Push, SW61 SW_Push, SW62 SW_Push, SW63 SW_Push, SW64 SW_Push, SW65 SW_Push, SW66 SW_Push, SW67 SW_Push, SW68 SW_Push, SW69 SW_Push, SW7 SW_Push, SW8 SW_Push, SW9 SW_Push, U1 ATmega32U4-A, Y1 16MHz

Commit message: fix manually where the kbplace autorouter failed
Routing:
- net ROW4: track 142.9 -> 286.0 mm
- net ROW2: track 216.7 -> 281.9 mm
- net ROW0: track 228.6 -> 288.8 mm
- net ROW3: track 242.9 -> 275.3 mm
- net COL1: track 67.0 -> 94.1 mm
- net COL13: track 60.1 -> 86.8 mm
- net COL10: track 86.0 -> 87.9 mm
- net COL9: track 86.0 -> 87.9 mm
- net COL5: track 87.0 -> 88.9 mm
- net COL2: track 89.0 -> 90.8 mm
- net COL0: track 83.1 -> 84.9 mm
- net COL14: track 76.2 -> 77.9 mm
- net COL12: track 84.1 -> 85.7 mm
- net COL8: track 67.0 -> 68.4 mm
- net COL6: track 67.0 -> 68.4 mm
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
Commit message: sort of arrange the mcu related components
need to get the pcb outline next to do proper positioning.
Parts:
- C1, C2, C3, C4, C7, C8, F1, J1, R1, R2, R3, R4, R5, R6, SW69, U1, USB1, Y1: moved to B.Cu
- C5, C6: value C_Small -> 22pF; moved to B.Cu
- moved C1 371.5 mm to (219.9, 221.8), turned to 90 degrees
- moved R1 369.5 mm to (237.7, 205.9), turned to -90 degrees
- moved C5 365.5 mm to (227.1, 218.2), turned to 180 degrees
- moved C4 362.0 mm to (215.5, 221.8), turned to -90 degrees
- moved C2 361.9 mm to (221.3, 209.9)
- moved C6 357.5 mm to (228.3, 208.3), turned to -90 degrees
- moved SW69 353.1 mm to (240.8, 211.2)
- moved R4 353.0 mm to (207.2, 221.6), turned to 180 degrees
- moved J1 351.7 mm to (238.8, 191.4), turned to 90 degrees
- moved C3 346.1 mm to (208.0, 203.9)
- moved C7 344.3 mm to (217.3, 203.8), turned to 180 degrees
- moved Y1 340.2 mm to (227.1, 214.1), turned to 90 degrees
- moved C8 337.9 mm to (213.2, 201.8), turned to 90 degrees
- moved R2 334.4 mm to (210.4, 186.6), turned to 90 degrees
- moved R3 333.9 mm to (212.6, 186.6), turned to 90 degrees
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Routing:
- net Net-(U1-XTAL2): track 0.00 -> 13.8 mm, vias 0 -> 2
- net Net-(USB1-CC2): track 0.00 -> 13.5 mm
- net Net-(D69-I/O2): track 0.00 -> 13.2 mm
- net Net-(D69-I/O1): track 0.00 -> 13.2 mm
- net Net-(U1-XTAL1): track 0.00 -> 13.1 mm
- net +5V: track 0.00 -> 9.94 mm
- net Net-(USB1-CC1): track 0.00 -> 9.03 mm
- net Net-(D69-VCC): track 0.00 -> 7.75 mm
- net Net-(U1-UCAP): track 0.00 -> 4.14 mm
- net GND: track 0.00 -> 2.65 mm

Commit message: adjust horizontal matrix row traces location
Parts:
- moved C1 44.4 mm to (191.5, 187.6)
- moved C5 44.4 mm to (198.7, 184.1)
- moved R1 44.4 mm to (209.3, 171.8)
- moved R2 44.4 mm to (182.0, 152.4)
- moved R3 44.4 mm to (184.2, 152.4)
- moved R4 44.4 mm to (178.8, 187.4)
- moved R5 44.4 mm to (174.0, 143.1)
- moved R6 44.4 mm to (174.0, 145.4)
- moved USB1 44.4 mm to (183.1, 134.7)
- moved Y1 44.4 mm to (198.7, 179.9)
- moved SW69 44.4 mm to (212.4, 177.0)
- moved C3 44.4 mm to (179.6, 169.8)
- moved C4 44.4 mm to (187.1, 187.7)
- moved C8 44.4 mm to (184.8, 167.7)
- moved F1 44.4 mm to (188.2, 149.2)
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Routing:
- net Net-(D69-VCC): track 7.75 -> 2.65 mm
- net ROW2: track 281.9 -> 278.6 mm
- net ROW0: track 288.8 -> 285.8 mm
- net ROW4: track 286.0 -> 283.4 mm
- net COL1: track 94.1 -> 96.2 mm
- net ROW3: track 275.3 -> 273.8 mm
- net Net-(D14-A): track 8.22 -> 6.95 mm
- net Net-(D62-A): track 8.22 -> 6.95 mm
- net Net-(D41-A): track 8.22 -> 6.95 mm
- net Net-(D36-A): track 8.22 -> 6.95 mm
- net Net-(D8-A): track 8.22 -> 6.95 mm
- net Net-(D64-A): track 8.22 -> 6.95 mm
- net Net-(D25-A): track 8.22 -> 6.95 mm
- net Net-(D52-A): track 8.22 -> 6.95 mm
- net Net-(D33-A): track 8.22 -> 6.95 mm
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
Commit message: roughly position mcu and sourrounding components
Also change to different usbc footprint
Parts:
- C3, C4, C7, C8, R4: moved to F.Cu
- USB1: footprint ai03-2725_Type-C:USB_C_GCT_USB4085 -> Connector_USB:USB_C_Receptacle_HRO_TYPE-C-31-M-12
- moved D69 175.3 mm to (73.1, 82.6), turned to 180 degrees
- moved SW69 167.9 mm to (58.9, 108.9), turned to 90 degrees
- moved R1 165.4 mm to (54.7, 113.0), turned to 90 degrees
- moved J1 153.0 mm to (61.7, 120.8), turned to 180 degrees
- moved C6 133.0 mm to (83.5, 109.9)
- moved C5 132.8 mm to (90.3, 107.5), turned to -90 degrees
- moved Y1 132.0 mm to (86.9, 109.8), turned to -90 degrees
- moved R3 130.2 mm to (72.1, 86.2)
- moved C1 129.8 mm to (82.7, 116.8), turned to -90 degrees
- moved F1 127.6 mm to (77.4, 86.0)
- moved R2 126.6 mm to (74.1, 86.2)
- moved R5 125.9 mm to (64.0, 81.9)
- moved R6 125.9 mm to (64.0, 84.2)
- moved USB1 125.6 mm to (73.1, 73.9)
- moved C2 123.2 mm to (84.8, 116.8), turned to 90 degrees
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Connections:
- net Net-(D69-I/O1) renamed /DR+
- net Net-(D69-I/O2) renamed /DR-
Routing:
- net +5V: track 9.94 -> 60.2 mm, vias 0 -> 6
- net /D-: track 0.00 -> 45.8 mm
- net /D+: track 0.00 -> 45.0 mm
- net Net-(J1-~{RST}): track 0.00 -> 41.6 mm, vias 0 -> 1
- net ROW1: track 281.0 -> 257.2 mm
- net /MOSI: track 0.00 -> 23.4 mm, vias 0 -> 1
- net /MISO: track 0.00 -> 20.5 mm, vias 0 -> 1
- net /SCK: track 0.00 -> 20.2 mm, vias 0 -> 1
- net Net-(USB1-CC2): track 13.5 -> 0.00 mm
- net Net-(D69-VCC): track 2.65 -> 13.2 mm, vias 0 -> 2
- net Net-(USB1-CC1): track 9.03 -> 0.00 mm
- net Net-(D16-A): track 6.95 -> 2.56 mm
- net /DR-: track 13.2 -> 9.41 mm
- net Net-(U1-XTAL2): track 13.8 -> 10.8 mm, vias 2 -> 0
- net GND: track 2.65 -> 0.00 mm
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- added copper zone on B.Cu, net GND
- added copper zone on F.Cu, net GND
Other:
- board outline added: 321.8 x 119.6 mm

Commit message: set outline and fix position of mcu, connectors etc.
next step is routing the rows/column connections to mcu
Parts:
- removed D69: PRTR5V0U2X, Package_TO_SOT_SMD:SOT-143
- removed F1: 500m, Fuse:Fuse_1206_3216Metric_Pad1.42x1.75mm_HandSolder
- removed R2, R3: 22, Resistor_SMD:R_0805_2012Metric_Pad1.20x1.40mm_HandSolder
- removed R5, R6: 5.1k, Resistor_SMD:R_0805_2012Metric_Pad1.20x1.40mm_HandSolder
- removed USB1: GCT USB-C USB4085-GF-A, Connector_USB:USB_C_Receptacle_HRO_TYPE-C-31-M-12
- added D71: PRTR5V0U2X, Package_TO_SOT_SMD:SOT-143, B.Cu at (75.6, 93.5)
- added F2: 500m, Fuse:Fuse_1206_3216Metric_Pad1.42x1.75mm_HandSolder, B.Cu at (83.7, 90.3)
- added J2: USB4105GFA120, kbd_custom:GCT_USB4105GFA120, B.Cu at (75.6, 84.6)
- added R11: 22, Resistor_SMD:R_0805_2012Metric_Pad1.20x1.40mm_HandSolder, B.Cu at (74.6, 97.6)
- added R12: 22, Resistor_SMD:R_0805_2012Metric_Pad1.20x1.40mm_HandSolder, B.Cu at (76.6, 97.6)
- added R15: 5.1k, Resistor_SMD:R_0805_2012Metric_Pad1.20x1.40mm_HandSolder, F.Cu at (74.3, 85.6)
- added R16: 5.1k, Resistor_SMD:R_0805_2012Metric_Pad1.20x1.40mm_HandSolder, F.Cu at (77.0, 85.6)
- moved R1 8.38 mm to (60.7, 118.8), turned to 180 degrees
- moved D68 6.69 mm to (353.3, 177.9), turned to 0 degrees
- moved D15 6.69 mm to (353.3, 101.7), turned to 0 degrees
- moved D30 6.69 mm to (353.3, 120.7), turned to 0 degrees
- moved D44 6.69 mm to (353.3, 139.8), turned to 0 degrees
- moved D58 6.69 mm to (353.3, 158.8), turned to 0 degrees
- moved J1 5.43 mm to (64.5, 125.5)
- moved SW69 5.43 mm to (61.7, 113.5)
- moved C5 4.70 mm to (87.0, 104.1), turned to 0 degrees
- moved D1 4.70 mm to (69.5, 101.1)
- moved D17 2.31 mm to (103.9, 116.4), turned to 180 degrees
- moved Y1 1.70 mm to (86.9, 108.1)
- moved C6 1.70 mm to (83.5, 108.2)
Routing:
- net +5V: track 60.2 -> 101.5 mm
- net ROW1: track 257.2 -> 292.8 mm, vias 0 -> 2
- net Net-(D71-VCC): track 0.00 -> 13.7 mm, vias 0 -> 2
- net Net-(D69-VCC): track 13.2 -> 0.00 mm, vias 2 -> 0
- net /D+: track 45.0 -> 32.5 mm
- net /D-: track 45.8 -> 33.2 mm
- net GND: track 0.00 -> 10.2 mm, vias 0 -> 18
- net ROW3: track 273.8 -> 266.6 mm
- net ROW2: track 278.6 -> 271.4 mm
- net ROW4: track 283.4 -> 276.1 mm
- net Net-(J1-~{RST}): track 41.6 -> 48.1 mm
- net Net-(U1-XTAL1): track 14.5 -> 18.1 mm
- net Net-(J2-CC2): track 0.00 -> 2.92 mm, vias 0 -> 1
- net Net-(J2-CC1): track 0.00 -> 2.80 mm, vias 0 -> 1
- net Net-(U1-XTAL2): track 10.8 -> 13.3 mm
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Other:
- board size 321.8 x 119.6 mm -> 305 x 102.8 mm

Commit message: adjust lower edge cut position for more clearance to stabilizer holes
Other:
- board size 305 x 102.8 mm -> 305 x 103.4 mm
Changed lines of the file:
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@@
 		(tags "SOD-123")
 		(property "Reference" "D15"
-			(at 0 2 360)
+			(at 0 2 0)
 			(layer "B.SilkS")
 			(effects
@@
 		)
 		(property "Value" "D"
-			(at 0 -2.1 360)
+			(at 0 -2.1 0)
 			(layer "B.Fab")
 			(effects
@@
 		)
 		(fp_text user "${REFERENCE}"
-			(at 0 2 360)
+			(at 0 2 0)
 			(layer "B.Fab")
 			(effects
@@
 		(tags "SOD-123")
 		(property "Reference" "D44"
-			(at 0 2 360)
+			(at 0 2 0)
 			(layer "B.SilkS")
 			(effects
@@
 		)
 		(property "Value" "D"
-			(at 0 -2.1 360)
+			(at 0 -2.1 0)
 			(layer "B.Fab")
 			(effects
@@
 		)
 		(fp_text user "${REFERENCE}"
-			(at 0 2 360)
+			(at 0 2 0)
 			(layer "B.Fab")
 			(effects
@@
 		(tags "capacitor handsolder")
 		(property "Reference" "C5"
-			(at 0 1.68 360)
+			(at 0 1.68 0)
 			(layer "B.SilkS")
 			(effects
@@
 		)
 		(property "Value" "22pF"
-			(at 0 -1.68 360)
+			(at 0 -1.68 0)
 			(layer "B.Fab")
 			(effects
@@
 		)
 		(fp_text user "${REFERENCE}"
-			(at 0 0 360)
+			(at 0 0 0)
 			(layer "B.Fab")
 			(effects
@@
 		(tags "SOD-123")
 		(property "Reference" "D30"
-			(at 0 2 360)
+			(at 0 2 0)
 			(layer "B.SilkS")
 			(effects
@@
 		)
 		(property "Value" "D"
-			(at 0 -2.1 360)
+			(at 0 -2.1 0)
 			(layer "B.Fab")
 			(effects
@@
 		)
 		(fp_text user "${REFERENCE}"
-			(at 0 2 360)
+			(at 0 2 0)
 			(layer "B.Fab")
 			(effects
@@
 		(tags "resistor handsolder")
 		(property "Reference" "R11"
-			(at 0 1.65 270)
+			(at 0 1.65 -90)
 			(layer "B.SilkS")
 			(effects
@@
 		)
 		(property "Value" "22"
-			(at 0 -1.65 270)
+			(at 0 -1.65 -90)
 			(layer "B.Fab")
 			(effects
@@
 		)
 		(fp_text user "${REFERENCE}"
-			(at 0 0 270)
+			(at 0 0 -90)
 			(layer "B.Fab")
 			(effects
@@
 		)
 		(fp_text user "${REFERENCE}"
-			(at 0 0 270)
+			(at 0 0 -90)
 			(layer "B.Fab")
 			(effects
@@
 		(tags "SOD-123")
 		(property "Reference" "D58"
-			(at 0 2 360)
+			(at 0 2 0)
 			(layer "B.SilkS")
 			(effects
@@
 		)
 		(property "Value" "D"
-			(at 0 -2.1 360)
+			(at 0 -2.1 0)
 			(layer "B.Fab")
 			(effects
@@
 		)
 		(fp_text user "${REFERENCE}"
-			(at 0 2 360)
+			(at 0 2 0)
 			(layer "B.Fab")
 			(effects
@@
 		(tags "resistor handsolder")
 		(property "Reference" "R12"
-			(at 0 1.65 270)
+			(at 0 1.65 -90)
 			(layer "B.SilkS")
 			(effects
@@
 		)
 		(property "Value" "22"
-			(at 0 -1.65 270)
+			(at 0 -1.65 -90)
 			(layer "B.Fab")
 			(effects
@@
 		)
 		(fp_text user "${REFERENCE}"
-			(at 0 0 270)
+			(at 0 0 -90)
 			(layer "B.Fab")
 			(effects
@@
 		(tags "fuse handsolder")
 		(property "Reference" "F2"
-			(at 0 1.82 360)
+			(at 0 1.82 0)
 			(layer "B.SilkS")
 			(effects
@@
 		)
 		(property "Value" "500m"
-			(at 0 -1.82 360)
+			(at 0 -1.82 0)
 			(layer "B.Fab")
 			(effects
@@
 		)
 		(fp_text user "${REFERENCE}"
-			(at 0 0 360)
+			(at 0 0 0)
 			(layer "B.Fab")
 			(effects
@@
 		(at 75.62875 84.565)
 		(property "Reference" "J2"
-			(at -1.825 8.635 360)
+			(at -1.825 8.635 0)
 			(layer "B.SilkS")
 			(effects
@@
 		)
 		(property "Value" "USB4105GFA120"
-			(at 5.795 7.135 360)
+			(at 5.795 7.135 0)
 			(layer "B.Fab")
 			(effects
@@
 		)
 		(fp_text user "PCB EDGE"
-			(at 5.4 -2.5 360)
+			(at 5.4 -2.5 0)
 			(layer "B.Fab")
 			(effects
@@
 		(tags "SOD-123")
 		(property "Reference" "D68"
-			(at 0 2 360)
+			(at 0 2 0)
 			(layer "B.SilkS")
 			(effects
@@
 		)
 		(property "Value" "D"
-			(at 0 -2.1 360)
+			(at 0 -2.1 0)
 			(layer "B.Fab")
 			(effects
@@
 		)
 		(fp_text user "${REFERENCE}"
-			(at 0 2 360)
+			(at 0 2 0)
 			(layer "B.Fab")
 			(effects
@@
 	)
 	(gr_arc
-		(start 58.47875 184.765)
-		(mid 57.064536 184.179214)
-		(end 56.47875 182.765)
+		(start 58.47875 185.342)
+		(mid 57.064504 184.756231)
+		(end 56.47875 183.342)
 		(stroke
 			(width 0.05)
@@
 	)
 	(gr_line
-		(start 58.47875 184.765)
-		(end 359.47875 184.765)
+		(start 58.47875 185.342)
+		(end 359.47875 185.342)
 		(stroke
 			(width 0.05)
@@
 	)
 	(gr_arc
-		(start 361.47875 182.765)
-		(mid 360.892964 184.179214)
-		(end 359.47875 184.765)
-		(locked yes)
+		(start 361.47875 183.342)
+		(mid 360.892961 184.756196)
+		(end 359.47875 185.342)
 		(stroke
 			(width 0.05)
@@
 	(gr_line
 		(start 56.47875 89.865)
-		(end 56.47875 182.765)
+		(end 56.47875 183.342)
 		(stroke
 			(width 0.05)
@@
 	)
 	(gr_line
-		(start 361.47875 182.765)
+		(start 361.47875 183.342)
 		(end 361.47875 89.865)
-		(locked yes)
 		(stroke
 			(width 0.05)
@@
 	)
 	(segment
-		(start 82.17875 96.665)
-		(end 82.17875 99.265)
+		(start 82.87875 124.865)
+		(end 83.24875 124.495)
 		(width 0.5)
 		(layer "B.Cu")
@@
 	)
 	(segment
-		(start 91.57875 130.24)
-		(end 91.57875 131.365)
+		(start 82.17875 96.665)
+		(end 82.17875 99.265)
 		(width 0.5)
 		(layer "B.Cu")
@@
 	)
 	(segment
-		(start 85.17875 121.265)
-		(end 85.17875 119.965)
+		(start 91.57875 130.24)
+		(end 91.57875 131.365)
 		(width 0.5)
 		(layer "B.Cu")
@@
 	)
 	(segment
-		(start 82.87875 124.865)
-		(end 83.97875 123.765)
+		(start 82.67875 117.8025)
+		(end 81.51625 117.8025)
 		(width 0.5)
 		(layer "B.Cu")
@@
 	)
 	(segment
-		(start 82.67875 117.8025)
-		(end 81.51625 117.8025)
+		(start 82.61625 117.865)
+		(end 82.67875 117.8025)
 		(width 0.5)
 		(layer "B.Cu")
@@
 	)
 	(segment
-		(start 82.61625 117.865)
-		(end 82.67875 117.8025)
+		(start 83.24875 124.495)
+		(end 83.24875 123.195)
 		(width 0.5)
 		(layer "B.Cu")
@@
 	)
 	(segment
+		(start 85.17875 121.265)
+		(end 85.17875 119.965)
+		(width 0.5)
+		(layer "B.Cu")
+		(net 2)
+	)
+	(segment
 		(start 61.67875 125.165)
 		(end 61.985 125.47125)
@@
 	)
 	(segment
-		(start 83.97875 123.765)
-		(end 83.97875 122.465)
+		(start 83.24875 123.195)
+		(end 85.17875 121.265)
 		(width 0.5)
 		(layer "B.Cu")
@@
 		(width 0.5)
 		(layer "B.Cu")
-		(net 2)
-	)
-	(segment
-		(start 83.97875 122.465)
-		(end 85.17875 121.265)
-		(width 0.5)
-		(layer "B.Cu")
