File: pcb/hmkb65alps.kicad_pcb (KiCad board)
At the start: 2 copper layers, 305 x 103.4 mm, 157 parts, among them J1 AVR-ISP-6, J2 USB4105GFA120, SW1 SW_Push, SW10 SW_Push, SW11 SW_Push, SW12 SW_Push, SW13 SW_Push, SW14 SW_Push, SW15 SW_Push, SW16 SW_Push, SW17 SW_Push, SW18 SW_Push, SW19 SW_Push, SW2 SW_Push, SW20 SW_Push, SW21 SW_Push, SW22 SW_Push, SW23 SW_Push, SW24 SW_Push, SW25 SW_Push, SW26 SW_Push, SW27 SW_Push, SW28 SW_Push, SW29 SW_Push, SW3 SW_Push, SW30 SW_Push, SW31 SW_Push, SW32 SW_Push, SW33 SW_Push, SW34 SW_Push, SW35 SW_Push, SW36 SW_Push, SW37 SW_Push, SW38 SW_Push, SW39 SW_Push, SW4 SW_Push, SW40 SW_Push, SW41 SW_Push, SW42 SW_Push, SW43 SW_Push, SW44 SW_Push, SW45 SW_Push, SW46 SW_Push, SW47 SW_Push, SW48 SW_Push, SW49 SW_Push, SW5 SW_Push, SW50 SW_Push, SW51 SW_Push, SW52 SW_Push, SW53 SW_Push, SW54 SW_Push, SW55 SW_Push, SW56 SW_Push, SW57 SW_Push, SW58 SW_Push, SW59 SW_Push, SW6 SW_Push, SW60 SW_Push, SW61 SW_Push, SW62 SW_Push, SW63 SW_Push, SW64 SW_Push, SW65 SW_Push, SW66 SW_Push, SW67 SW_Push, SW68 SW_Push, SW69 SW_Push, SW7 SW_Push, SW8 SW_Push, SW9 SW_Push, U1 ATmega32U4-A, Y1 16MHz

Commit message: route and assign all rows/columns of the matrix
also add some more vias where found neccessary
Parts:
- moved D45 2.67 mm to (83.7, 158.0), turned to 180 degrees
Connections:
- U1 pad 12: unconnected-(U1-PB7-Pad12) -> ROW0
- U1 pad 18: unconnected-(U1-PD0-Pad18) -> COL1
- U1 pad 19: unconnected-(U1-PD1-Pad19) -> ROW1
- U1 pad 20: unconnected-(U1-PD2-Pad20) -> COL4
- U1 pad 21: unconnected-(U1-PD3-Pad21) -> COL2
- U1 pad 22: unconnected-(U1-PD5-Pad22) -> COL3
- U1 pad 25: unconnected-(U1-PD4-Pad25) -> COL5
- U1 pad 26: unconnected-(U1-PD6-Pad26) -> COL6
- U1 pad 27: unconnected-(U1-PD7-Pad27) -> COL7
- U1 pad 28: unconnected-(U1-PB4-Pad28) -> COL8
- U1 pad 29: unconnected-(U1-PB5-Pad29) -> COL9
- U1 pad 30: unconnected-(U1-PB6-Pad30) -> COL10
- U1 pad 31: unconnected-(U1-PC6-Pad31) -> COL11
- U1 pad 32: unconnected-(U1-PC7-Pad32) -> COL12
- U1 pad 36: unconnected-(U1-PF7-Pad36) -> COL13
- U1 pad 37: unconnected-(U1-PF6-Pad37) -> COL14
- U1 pad 38: unconnected-(U1-PF5-Pad38) -> ROW3
- U1 pad 39: unconnected-(U1-PF4-Pad39) -> ROW4
- U1 pad 40: unconnected-(U1-PF1-Pad40) -> ROW2
- U1 pad 41: unconnected-(U1-PF0-Pad41) -> COL0
Routing:
- net COL14: track 78.0 -> 349.6 mm, vias 0 -> 1
- net COL13: track 85.8 -> 326.1 mm, vias 0 -> 1
- net COL12: track 85.4 -> 310.0 mm, vias 0 -> 1
- net COL11: track 85.3 -> 276.0 mm, vias 0 -> 1
- net COL10: track 87.9 -> 258.8 mm, vias 0 -> 1
- net COL9: track 87.7 -> 238.8 mm, vias 0 -> 1
- net COL8: track 68.3 -> 200.1 mm, vias 0 -> 1
- net COL7: track 68.2 -> 181.1 mm, vias 0 -> 1
- net COL6: track 68.3 -> 162.0 mm, vias 0 -> 1
- net COL5: track 89.1 -> 163.6 mm, vias 0 -> 1
- net COL4: track 68.3 -> 127.5 mm, vias 0 -> 1
- net ROW4: track 276.1 -> 323.0 mm
- net COL3: track 68.2 -> 106.6 mm, vias 0 -> 1
- net ROW3: track 266.6 -> 294.8 mm
- net COL0: track 86.0 -> 107.6 mm, vias 0 -> 1
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
Commit message: add vias around outline
Routing:
- net GND: vias 82 -> 394

Commit message: add stitching vias
Routing:
- net GND: vias 394 -> 761
