File: plate/plate.kicad_pcb (KiCad board)
At the start: 2 copper layers, 317.8 x 114.6 mm, 0 parts

Commit message: come up with a plate that "should" work
Other:
- outline, holes or cut-outs redrawn
- board text added: "Plate outline should be on edge cut layer and locked. Use the (locked) key positions here to align the hole pattern on the edge cut layer. Mainly this is to easily swap to different stabilizer cutout variations. Import the pattern from dxf generated with yet-another-keyboard- builder."

Commit message: stitch planes because why not and reduce copper to edge clearance
Routing:
- net GND: vias 0 -> 1519
- added copper zone on B.Cu, net GND
- added copper zone on F.Cu, net GND
- removed copper zone on B.Cu, net (none)
- removed copper zone on F.Cu, net (none)
